Commit message: feat: refine calibration UI and optimize camera performance
- Moved calibration module to bottom of sidebar and changed default tab
- Disabled expensive MJPEG corner detection unless in calibration mode
- Added debounce to calibration mode toggle to fix React StrictMode race condition
- Throttled OpenCV corner detection in live feed to 2fps with 0.5s visual cache
- Filtered uvicorn logs from frontend console view
- Cleaned up spray gun from base CR5 robot URDF model
- Exposed sample calculation stats (used vs total) in calibration results UI

File: app/urdf/cr5_robot_with_gun.urdf (robot description, URDF)
Before this commit: robot cr5_robot, 10 links, 9 joints
Links:
- added link spray_gun; collision mesh filename=package://dobot_rviz/meshes/dobot_gazebo_sim/spray_gun.stl scale=0.001 0.001 0.001; visual mesh filename=package://dobot_rviz/meshes/dobot_gazebo_sim/spray_gun.stl scale=0.001 0.001 0.001
- added link spray_nozzle_link
Joints:
- added joint Link6_to_spray_gun: type fixed, parent Link6, child spray_gun, origin xyz=0 0 0 rpy=0 0 1.5708
- added joint Link6_to_spray_nozzle_link: type fixed, parent Link6, child spray_nozzle_link, origin xyz=0.002022 -0.0353263 0.3122347 rpy=0.0329936 -0.0038327 -2.3392176
