Commit message: feat(robot): integrate Viterbi DP into POI optimizer, align CLI/Web table diagnostics, and enforce 10% robot speed protection
- Refactor poi_optimizer.py to wrap SprayWaypointOptimizer (Viterbi DP global MoveL continuous optimization) with attached dense trajectory points (trajectory_q, trajectory_tcp)
- Unlock J1 physical limits to +/- 6.28 rad (+/- 360 deg) in URDF and kinematics for multi-turn unwrapping
- Set Home pose [90, 0, 90] and [20, 20, 180] deg tolerance envelope as default POI configuration in frontend and backend
- Add pixel-perfect ASCII table formatter with CJK visual width alignment in poi_optimizer.py and path_opt_cli.py
- Fix Web Console rendering in ConsoleLogZone.tsx with monospace <pre> blocks and horizontal scrolling for multi-line tables
- Enforce 10% speed factor, MoveL (SpeedL/AccL=10) and MoveJ (SpeedJ/AccJ=10) speed protection upon connecting real robot

File: app/urdf/cr5_robot.urdf (robot description, URDF)
Before this commit: robot cr5_robot, 10 links, 9 joints
Joints:
- joint joint1: limit lower=-3.14 upper=3.14 effort=100 velocity=3.14 -> lower=-6.28 upper=6.28 effort=100 velocity=3.14

File: app/urdf/cr5_robot_with_gun.urdf (robot description, URDF)
Before this commit: robot cr5_robot, 12 links, 11 joints
Joints:
- joint joint1: limit lower=-3.14 upper=3.14 effort=100 velocity=3.14 -> lower=-6.28 upper=6.28 effort=100 velocity=3.14
