Commit message: feat(tool): modularize composite end-effector parts with URDF material styling and automatic alignment tool

File: app/urdf/cr5_robot_with_my_tools.urdf (robot description, URDF)
Before this commit: robot cr5_robot, 12 links, 11 joints
Links:
- removed link my_tools
- added link my_tools_black; collision mesh filename=package://dobot_rviz/meshes/dobot_gazebo_sim/my_tools_black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 scale=0.001 0.001 0.001; visual mesh filename=package://dobot_rviz/meshes/dobot_gazebo_sim/my_tools_black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 scale=0.001 0.001 0.001
- added link my_tools_fingers; collision mesh filename=package://dobot_rviz/meshes/dobot_gazebo_sim/my_tools_finge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 scale=0.001 0.001 0.001; visual mesh filename=package://dobot_rviz/meshes/dobot_gazebo_sim/my_tools_finge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 scale=0.001 0.001 0.001
- added link my_tools_nozzle; collision mesh filename=package://dobot_rviz/meshes/dobot_gazebo_sim/my_tools_nozzl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 scale=0.001 0.001 0.001; visual mesh filename=package://dobot_rviz/meshes/dobot_gazebo_sim/my_tools_nozzl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 scale=0.001 0.001 0.001
- added link my_tools_silver; collision mesh filename=package://dobot_rviz/meshes/dobot_gazebo_sim/my_tools_silve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 scale=0.001 0.001 0.001; visual mesh filename=package://dobot_rviz/meshes/dobot_gazebo_sim/my_tools_silve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 scale=0.001 0.001 0.001
Joints:
- removed joint Link6_to_my_tools
- added joint Link6_to_my_tools_black: type fixed, parent Link6, child my_tools_black, origin xyz=0 0 0 rpy=0 0 1.5708
- added joint Link6_to_my_tools_fingers: type fixed, parent Link6, child my_tools_fingers, origin xyz=0 0 0 rpy=0 0 1.5708
- added joint Link6_to_my_tools_nozzle: type fixed, parent Link6, child my_tools_nozzle, origin xyz=0 0 0 rpy=0 0 1.5708
- added joint Link6_to_my_tools_silver: type fixed, parent Link6, child my_tools_silver, origin xyz=0 0 0 rpy=0 0 1.5708

Commit message: fixed urdf tools direction

File: app/urdf/cr5_robot_with_my_tools.urdf (robot description, URDF)
Before this commit: robot cr5_robot, 15 links, 14 joints
Joints:
- joint Link6_to_my_tools_black: origin xyz=0 0 0 rpy=0 0 1.5708 -> xyz=0 0 0 rpy=0 0 -1.5708
- joint Link6_to_my_tools_fingers: origin xyz=0 0 0 rpy=0 0 1.5708 -> xyz=0 0 0 rpy=0 0 -1.5708
- joint Link6_to_my_tools_nozzle: origin xyz=0 0 0 rpy=0 0 1.5708 -> xyz=0 0 0 rpy=0 0 -1.5708
- joint Link6_to_my_tools_silver: origin xyz=0 0 0 rpy=0 0 1.5708 -> xyz=0 0 0 rpy=0 0 -1.5708
- joint Link6_to_spray_nozzle_link: origin xyz=0.002022 -0.0353263 0.3122347 rpy=0.0329936 -0.0038327 -2.3392176 -> xyz=-0.002022 0.0353263 0.3122347 rpy=0.0329936 -0.0038327 0.8023751

Commit message: feat(interactive): 添加SAM分割标签支持和改进路径验证功能
- 在MaskData类型中添加labels字段用于存储分割标签信息
- 实现前端交互式操作中标签数据的传递和保存功能
- 优化路径验证服务中的POI约束配置逻辑
- 添加锚点来源配置选项包括config、home、live和raw模式
- 实现机械臂工具坐标系自动切换功能
- 增加重建服务的子进程隔离机制防止崩溃影响主进程
- 改进SAM服务中点数据解析支持标签信息提取
- 添加钧舵夹爪硬件控制模块和Modbus通信支持
- 优化模板保存时的掩码数据处理流程

File: app/urdf/cr5_robot_with_my_tools.urdf (robot description, URDF)
Before this commit: robot cr5_robot, 15 links, 14 joints
Links:
- removed link my_tools_nozzle
- removed link spray_nozzle_link
- added link gripper_tip_link
- added link laser_head_link
- added link my_tools_laser_nozzle; collision mesh filename=package://dobot_rviz/meshes/dobot_gazebo_sim/my_tools_laser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 scale=0.001 0.001 0.001; visual mesh filename=package://dobot_rviz/meshes/dobot_gazebo_sim/my_tools_laser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 scale=0.001 0.001 0.001
Joints:
- removed joint Link6_to_my_tools_nozzle
- removed joint Link6_to_spray_nozzle_link
- added joint Link6_to_gripper_tip_link: type fixed, parent Link6, child gripper_tip_link, origin xyz=-0.003359 -0.022217 0.251675 rpy=0.0430748 0.0400553 3.0562138
- added joint Link6_to_laser_head_link: type fixed, parent Link6, child laser_head_link, origin xyz=0.002404 0.016223 0.138333 rpy=-0.0183085 -0.0662699 -1.4414342
- added joint Link6_to_my_tools_laser_nozzle: type fixed, parent Link6, child my_tools_laser_nozzle, origin xyz=0 0 0 rpy=0 0 -1.5708

Commit message: feat(robot): add articulated parallel gripper control, telemetry, and 3D simulation
- Decouple monolithic fingers mesh into independent left/right STLs via tools/split_gripper_mesh.py

- Define prismatic sliding joints for gripper in cr5_robot_with_my_tools.urdf

- Consolidate gripper hardware specs and fail-safe defaults in JunduoGripper driver

- Implement batch 3-register Modbus telemetry query and adaptive high-frequency polling

- Add REST/WebSocket APIs with disconnect interlock protection

- Support speed, clamp force, and stroke controls in JogControlPanel

- Add 60fps frame-level LERP interpolation in Robot3DViewer for smooth 3D opening/closing

File: app/urdf/cr5_robot_with_my_tools.urdf (robot description, URDF)
Before this commit: robot cr5_robot, 16 links, 15 joints
Links:
- removed link my_tools_fingers
- added link my_tools_finger_left; collision mesh filename=package://dobot_rviz/meshes/dobot_gazebo_sim/my_tools_finge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 scale=0.001 0.001 0.001; visual mesh filename=package://dobot_rviz/meshes/dobot_gazebo_sim/my_tools_finge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 scale=0.001 0.001 0.001
- added link my_tools_finger_right; collision mesh filename=package://dobot_rviz/meshes/dobot_gazebo_sim/my_tools_finge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 scale=0.001 0.001 0.001; visual mesh filename=package://dobot_rviz/meshes/dobot_gazebo_sim/my_tools_finge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 scale=0.001 0.001 0.001
Joints:
- removed joint Link6_to_my_tools_fingers
- added joint gripper_finger_left_joint: type prismatic, parent Link6, child my_tools_finger_left, origin xyz=0 0 0 rpy=0 0 -1.5708, axis 0 1 0, limit lower=0.0 upper=0.025 effort=60 velocity=0.1
- added joint gripper_finger_right_joint: type prismatic, parent Link6, child my_tools_finger_right, origin xyz=0 0 0 rpy=0 0 -1.5708, axis 0 -1 0, limit lower=0.0 upper=0.025 effort=60 velocity=0.1
